File: elec/main_board/main_board.kicad_sch (KiCad schematic)
At the start: 69 parts, among them J1 B2B-PH, J13 B4B-ZR(LF)(SN), J2 B2B-PH, J3 PSR-41253-06O, J4 PinHeader, J5 PSR-41253-06O, J6 PSR-41253-06O, J7 Conn_01x02, J8 PSR-41253-06O, Q1 IRLML6344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

Commit message: 再設計　部品配置完了
Signed-off-by: Kazuki Iida <elkel53930@gmail.com>
Parts:
- removed D9: SFH4550, Library:SFH4550_Mirror, symbol Device:LED
- removed J3: PSR-41253-06O, Connector_PinHeader_2.54mm:PinHeader_1x06_P2.54mm_Vertical, symbol Connector:Conn_01x06_Male
- removed J5, J8: PSR-41253-06O, Connector_PinHeader_2.54mm:PinHeader_1x06_P2.54mm_Vertical, symbol Connector:Conn_01x06_Female
- removed L1, L2: NR6045T100M, Inductor_SMD:L_Changjiang_FNR6040S, symbol Device:L
- removed Q12: ST-1KL3A, Library:ST-1KL3A_Mirror, symbol Device:Q_Photo_NPN_EC
- removed Q4: IRLML6344, Package_TO_SOT_SMD:SOT-23, symbol Transistor_FET:IRLML2060
- removed R13: 0603WAF1000T5E, Resistor_SMD:R_0603_1608Metric, symbol Device:R
- removed R17: 0603WAF1002T5E, Resistor_SMD:R_0603_1608Metric, symbol Device:R
- removed R9: 0603WAF4700T5E, Resistor_SMD:R_0603_1608Metric, symbol Device:R
- added H5: M2.6 mounting hole, Library:M2.6 Mounting Hole, symbol Mechanical:MountingHole
- added H6, H7: M3 mounting hole, MountingHole:MountingHole_3.2mm_M3, symbol Mechanical:MountingHole
- added J11: B7B-ZR, Connector_JST:JST_ZH_B7B-ZR_1x07_P1.50mm_Vertical, symbol Connector_Generic:Conn_01x07
- added J5: PSR-41253-06O, Connector_PinHeader_1.27mm:PinHeader_1x06_P1.27mm_Vertical, symbol Connector:Conn_01x06_Male
- added J8: Conn_01x07_Pin, Connector_PinHeader_1.27mm:PinHeader_1x07_P1.27mm_Vertical, symbol Connector:Conn_01x07_Pin
- J1, J2: value B2B-PH -> Motor; footprint Connector_JST:JST_PH_B2B-PH-K_1x02_P2.00mm_Vertical -> Connector_PinHeader_2.00mm:PinHeader_1x02_P2.00mm_Vertical
- J6: footprint Connector_PinHeader_2.54mm:PinHeader_1x06_P2.54mm_Vertical -> Connector_PinHeader_1.27mm:PinHeader_1x06_P1.27mm_Vertical
- U6: value ESP32-S3-WROOM-1 -> ESP32-S3-WROOM-1U; footprint RF_Module:ESP32-S3-WROOM-1 -> RF_Module:ESP32-S3-WROOM-1U
Connections:
- net RF_EN is gone; now on net SPI2_SCK: U6.33 (IO40)
- net RF_SEN is gone; now on net PWM_FAN: U6.38 (IO2)
- net +3V3: now also J11.1 (Pin_1)
- net BALL_DET: now also U6.22 (IO14); no longer U6.23 (IO21)
- net BAT_MON: now also U6.21 (IO13); no longer U6.8 (IO15)
- net CS_ENC_L: now also U6.17 (IO9), J11.6 (Pin_6); no longer U6.11 (IO18)
- net CS_ENC_R: now also U6.16 (IO46), J11.7 (Pin_7); no longer U6.26 (IO45)
- net CS_IMU: now also U6.34 (IO41); no longer U6.22 (IO14)
- net CWCCW_L: now also U6.24 (IO47); no longer U6.18 (IO10)
- net CWCCW_R: now also U6.26 (IO45); no longer U6.25 (IO48)
- net GND: now also J11.2 (Pin_2)
- net LED_0: now also U6.14 (USB_D+); no longer U6.15 (IO3)
- net LED_1: now also U6.15 (IO3); no longer U6.16 (IO46)
- net PWM_FAN: no longer U6.32 (IO39)
- net PWM_L: now also U6.23 (IO21); no longer U6.17 (IO9)
- net PWM_R: now also U6.25 (IO48); no longer U6.24 (IO47)
- net SERVO_SIG1: now also U6.39 (IO1); no longer U6.28 (IO35)
- net SPI1_MISO: now also U6.19 (IO11), J11.4 (Pin_4); no longer U6.13 (USB_D-)
- net SPI1_MOSI: now also U6.20 (IO12), J11.3 (Pin_3); no longer U6.14 (USB_D+)
- net SPI1_SCK: now also U6.18 (IO10), J11.5 (Pin_5); no longer U6.12 (IO8)
- net SPI2_MISO: now also U6.31 (IO38); no longer U6.19 (IO11)
- net SPI2_MOSI: now also U6.32 (IO39); no longer U6.20 (IO12)
- net SPI2_SCK: no longer U6.21 (IO13)
- net ENCL_CS_L: now reaches U9.1 (~{CS})
- net ENCL_CS_L: now also J8.6 (Pin_6)
- net ENCL__3V3: now reaches C15.2, U9.12 (VDD3V3)
- net ENCL__3V3: now also J5.1 (Pin_1), J8.1 (Pin_1)
- net ENCL_GND: now reaches C15.1, U9.13 (GND), U9.5 (TST)
- net ENCL_GND: now also J5.2 (Pin_2), J8.2 (Pin_2)
- net ENCL_SCK: now reaches U9.2 (CLK)
- net ENCL_SCK: now also J5.5 (Pin_5), J8.5 (Pin_5)
- net ENCL_MISO: now reaches U9.3 (MISO)
- net ENCL_MISO: now also J5.4 (Pin_4), J8.4 (Pin_4)
- net ENCL_MOSI: now reaches U9.4 (MOSI)
- net ENCL_MOSI: now also J5.3 (Pin_3), J8.3 (Pin_3)
- net at J1.2 (Pin_2): now also U2.4 (OUTB)
- net at U5.4 (OUTB): now also J2.2 (Pin_2)
- net L_SEN: now reaches U6.9 (IO16)
- net L_SEN: now also Q9.1 (E), R6.2
- net ENCR_CS_R: now reaches J6.6 (Pin_6), U10.1 (~{CS})
- net ENCR__3V3: now reaches C16.2, J6.1 (Pin_1), U10.12 (VDD3V3)
- net ENCR_GND: now reaches C16.1, J6.2 (Pin_2), U10.13 (GND), U10.5 (TST)
- net ENCR_SCK: now reaches J6.5 (Pin_5), U10.2 (CLK)
- net ENCR_MISO: now reaches J6.4 (Pin_4), U10.3 (MISO)
- net ENCR_MOSI: now reaches J6.3 (Pin_3), U10.4 (MOSI)
- net LF_EN renamed L_EN
- net L_EN: now also U6.8 (IO15); no longer U6.7 (IO7)
- removed net LF_SEN: Q9.1 (E), R6.2, U6.6 (IO6)
- net LS_EN renamed F_EN
- net F_EN: now also U6.6 (IO6); no longer U6.5 (IO5)
- net LS_SEN renamed F_SEN
- net F_SEN: now also U6.7 (IO7); no longer U6.4 (IO4)
- net RS_EN renamed R_EN
- net R_EN: now also U6.4 (IO4); no longer U6.34 (IO41)
- net RS_SEN renamed R_SEN
- net R_SEN: now also U6.5 (IO5); no longer U6.39 (IO1)
- new net ENCL_CS_R: J5.6 (Pin_6), J8.7 (Pin_7)
- no-connect marks 24 -> 25
Other:
- note added: "from Enc L"
- note added: "to Enc R"
- moved on the sheet: C15, C16, D6, D7, D8, J6, Q1, Q10, Q11, Q2, Q3, Q9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

Commit message: 配線作業中
Signed-off-by: Kazuki Iida <elkel53930@gmail.com>
Parts:
- removed C15: CC0603KRX7R9BB104, Capacitor_SMD:C_0402_1005Metric, symbol Device:C_Small
- removed C16: CL05B104KO5NNNC, Capacitor_SMD:C_0402_1005Metric, symbol Device:C_Small
- removed J5, J6: PSR-41253-06O, Connector_PinHeader_1.27mm:PinHeader_1x06_P1.27mm_Vertical, symbol Connector:Conn_01x06_Male
- removed J8: Conn_01x07_Pin, Connector_PinHeader_1.27mm:PinHeader_1x07_P1.27mm_Vertical, symbol Connector:Conn_01x07_Pin
- removed U10, U9: AS5047D, Package_SO:TSSOP-14_4.4x5mm_P0.65mm, symbol Sensor_Magnetic:AS5047D
- added C1, C2, C4: CL21A106KAYNNNE, Capacitor_SMD:C_0805_2012Metric, symbol Device:C_Small
- added R9: 0603WAF1002T5E, Resistor_SMD:R_0603_1608Metric, symbol Device:R
Connections:
- net +BATT: now also C1.2, C2.2, C4.2
- net CWCCW_R: now also R9.2
- net GND: now also C1.1, C2.1, C4.1, R9.1
- no-connect marks 25 -> 11
Other:
- note added: "Boot strap PullDown"
- note removed: "AS5047 SPI mode = 1 (Latch at fall edges)"
- note removed: "Encoders"
- note removed: "from Enc L"
- note removed: "to Enc R"
- moved on the sheet: D1, D6, D7, D8, J11, Q1, Q10, Q11, Q2, Q3, Q9, R1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
