File: elec/rpi_board/rpi_board.kicad_sch (KiCad schematic)
At the start: 30 parts, among them J1 B2B-ZR, J2 Conn_01x10, J3 PinHeader, J4 FH12-22S-0.5SH, J5 FSS-42085-03, J6 FSS-42085-03, Q1 IRLML6344, Q2 IRLML6344, U1 MCP3221, U2 74LVC1G07SE-7

Commit message: アートワーク完了、発注
Signed-off-by: Kazuki Iida <elkel53930@gmail.com>
Parts:
- added C8, C9: CC0603KRX7R9BB104, Capacitor_SMD:C_0603_1608Metric, symbol Device:C_Small
Connections:
- net +5V: now also C8.2, C9.2
- net GND: now also C8.1, C9.1
- net USB_DM renamed USB_D-
- net USB_DP renamed USB_D+
