File: elec/sub_boards/sub_boards.kicad_pcb (KiCad board)
At the start: 2 copper layers, 65.3 x 47.4 mm, 14 parts, among them J1 Conn_01x10, J5 PSR-41253-06O, J6 PSR-41253-06O, J8 Conn_01x07_Pin, SW1 TVBP06-B043CB-B, SW2 TVBP06-B043CB-B, U10 AS5047D, U9 AS5047D

Commit message: アートワーク完了、発注
Signed-off-by: Kazuki Iida <elkel53930@gmail.com>
Parts:
- added D3: BAS516, Diode_SMD:D_SOD-523, F.Cu at (176.6, 98.5)
- added LS1: SMT-0440-T-2-R, Library:SMT-0440-T-2-R, F.Cu at (173.1, 98.5)
Routing:
- net +3.3V: track 55.0 -> 61.4 mm
- net /BUZZER: track 10.7 -> 12.8 mm
