File: elec/sub_boards/sub_boards.kicad_sch (KiCad schematic)
At the start: 14 parts, among them J1 Conn_01x10, J5 PSR-41253-06O, J6 PSR-41253-06O, J8 Conn_01x07_Pin, SW1 TVBP06-B043CB-B, SW2 TVBP06-B043CB-B, U10 AS5047D, U9 AS5047D

Commit message: アートワーク完了、発注
Signed-off-by: Kazuki Iida <elkel53930@gmail.com>
Parts:
- added D3: BAS516, Diode_SMD:D_SOD-523, symbol Diode:BAS516
- added LS1: SMT-0440-T-2-R, Library:SMT-0440-T-2-R, symbol Device:Speaker
Connections:
- net +3.3V: now also D3.1 (K), LS1.1
- net BUZZER: now also D3.2 (A), LS1.2
Other:
- moved on the sheet: BZ1
