File: elec/sub_boards/sub_boards.kicad_sch (KiCad schematic)
At the start: 16 parts, among them J1 Conn_01x10, J5 PSR-41253-06O, J6 PSR-41253-06O, J8 Conn_01x07_Pin, SW1 TVBP06-B043CB-B, SW2 TVBP06-B043CB-B, U10 AS5047D, U9 AS5047D

Commit message: 新エンコーダ基板のアートワーク作業中
Signed-off-by: Kazuki Iida <elkel53930@gmail.com>
Parts:
- added H3, H4, H5, H6: M2, MountingHole:MountingHole_2.1mm, symbol Mechanical:MountingHole
- J5, J6: footprint Connector_PinHeader_1.27mm:PinHeader_1x06_P1.27mm_Vertical -> Connector_JST:JST_ZH_B6B-ZR_1x06_P1.50mm_Vertical
- J8: footprint Connector_PinHeader_1.27mm:PinHeader_1x07_P1.27mm_Vertical -> Connector_JST:JST_ZH_B7B-ZR_1x07_P1.50mm_Vertical
Connections:
- net ENCR_CS_R: now also J6.1 (Pin_1); no longer J6.6 (Pin_6)
- net ENCR_GND: now also J6.5 (Pin_5); no longer J6.2 (Pin_2)
- net ENCR_MISO: now also J6.3 (Pin_3); no longer J6.4 (Pin_4)
- net ENCR_MOSI: now also J6.4 (Pin_4); no longer J6.3 (Pin_3)
- net ENCR_SCK: no longer J6.5 (Pin_5)
- net ENCR__3V3: now also J6.6 (Pin_6); no longer J6.1 (Pin_1)

Commit message: 新しいエンコーダ基板のアートワーク官僚
Signed-off-by: Kazuki Iida <elkel53930@gmail.com>
Parts:
- C15: value CC0603KRX7R9BB104 -> ~; footprint Capacitor_SMD:C_0402_1005Metric -> Capacitor_SMD:C_0805_2012Metric_Pad1.18x1.45mm_HandSolder
- C16: value CL05B104KO5NNNC -> ~; footprint Capacitor_SMD:C_0402_1005Metric -> Capacitor_SMD:C_0805_2012Metric_Pad1.18x1.45mm_HandSolder
Connections:
- net ENCR_SCK: now also J6.2 (Pin_2)
Other:
- moved on the sheet: C16
Changed lines of the file:
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@@
-	(wire
-		(pts
-			(xy 189.23 113.03) (xy 215.9 113.03)
-		)
-		(stroke
-			(width 0)
-			(type default)
-		)
-	)
 	(wire
 		(pts
@@
 		(pts
 			(xy 87.63 104.14) (xy 91.44 104.14)
+		)
+		(stroke
+			(width 0)
+			(type default)
+		)
+	)
+	(wire
+		(pts
+			(xy 186.69 113.03) (xy 215.9 113.03)
 		)
 		(stroke
@@
 	(symbol
 		(lib_id "Device:C_Small")
-		(at 209.55 124.46 0)
-		(mirror x)
+		(at 209.55 124.46 180)
 		(unit 1)
 		(exclude_from_sim no)
@@
 		(dnp no)
 		(property "Reference" "C16"
-			(at 211.074 132.842 0)
+			(at 208.026 132.842 0)
 			(effects
 				(font
@@
 			)
 		)
-		(property "Value" "CL05B104KO5NNNC"
-			(at 205.74 132.08 90)
+		(property "Value" "~"
+			(at 213.36 132.08 90)
 			(effects
 				(font
@@
 			)
 		)
-		(property "Footprint" "Capacitor_SMD:C_0402_1005Metric"
+		(property "Footprint" "Capacitor_SMD:C_0805_2012Metric_Pad1.18x1.45mm_HandSolder"
 			(at 209.55 124.46 0)
 			(effects
@@
 			)
 		)
-		(property "Description" "0.1uF 50V X7R 1005"
+		(property "Description" "0.1uF 50V X7R 2012"
 			(at 209.55 131.064 0)
 			(effects
@@
 	)
 	(symbol
-		(lib_id "Device:C_Small")
-		(at 231.14 82.55 0)
-		(mirror x)
-		(unit 1)
-		(exclude_from_sim no)
-		(in_bom yes)
-		(on_board yes)
-		(dnp no)
-		(property "Reference" "C15"
-			(at 232.664 90.932 0)
-			(effects
-				(font
-					(size 1.27 1.27)
-				)
-				(justify right)
-			)
-		)
-		(property "Value" "CC0603KRX7R9BB104"
-			(at 227.33 90.17 90)
-			(effects
-				(font
-					(size 1.27 1.27)
-				)
-				(justify right)
-				(hide yes)
-			)
-		)
-		(property "Footprint" "Capacitor_SMD:C_0402_1005Metric"
-			(at 231.14 82.55 0)
-			(effects
-				(font
-					(size 1.27 1.27)
-				)
-				(hide yes)
-			)
-		)
-		(property "Datasheet" "~"
-			(at 231.14 82.55 0)
-			(effects
-				(font
-					(size 1.27 1.27)
-				)
-				(hide yes)
-			)
-		)
-		(property "Description" "0.1uF 50V X7R 1005"
-			(at 231.14 89.154 0)
-			(effects
-				(font
-					(size 1.27 1.27)
-				)
-			)
-		)
-		(property "フィールド4" ""
-			(at 231.14 82.55 0)
-			(effects
-				(font
-					(size 1.27 1.27)
-				)
-				(hide yes)
-			)
-		)
-		(pin "1"
-		)
-		(pin "2"
-		)
-		(instances
-			(project "sub_boards"
-				(path "/d5abadbb-7de1-45ef-bf83-ffcbea26f0f6"
-					(reference "C15")
-					(unit 1)
-				)
-			)
-		)
-	)
-	(symbol
 		(lib_id "Mechanical:MountingHole")
 		(at 256.54 146.05 0)
@@
 					(unit 1)
 				)
+			)
+		)
+	)
+	(symbol
+		(lib_id "Device:C_Small")
+		(at 231.14 82.55 0)
+		(mirror x)
+		(unit 1)
+		(exclude_from_sim no)
+		(in_bom yes)
+		(on_board yes)
+		(dnp no)
+		(property "Reference" "C15"
+			(at 232.664 90.932 0)
+			(effects
+				(font
+					(size 1.27 1.27)
+				)
+				(justify right)
+			)
+		)
+		(property "Value" "~"
+			(at 227.33 90.17 90)
+			(effects
+				(font
+					(size 1.27 1.27)
+				)
+				(justify right)
+				(hide yes)
+			)
+		)
+		(property "Footprint" "Capacitor_SMD:C_0805_2012Metric_Pad1.18x1.45mm_HandSolder"
+			(at 231.14 82.55 0)
+			(effects
+				(font
+					(size 1.27 1.27)
+				)
+				(hide yes)
+			)
+		)
+		(property "Datasheet" "~"
+			(at 231.14 82.55 0)
+			(effects
+				(font
+					(size 1.27 1.27)
+				)
+				(hide yes)
+			)
+		)
+		(property "Description" "0.1uF 50V X7R 2012"
+			(at 231.14 89.154 0)
+			(effects
+				(font
+					(size 1.27 1.27)
+				)
+			)
+		)
+		(property "フィールド4" ""
+			(at 231.14 82.55 0)
+			(effects
+				(font
+					(size 1.27 1.27)
+				)
+				(hide yes)
+			)
+		)
+		(pin "1"
+		)
+		(pin "2"
+		)
+		(instances
+			(project "sub_boards"
+				(path "/d5abadbb-7de1-45ef-bf83-ffcbea26f0f6"
+					(reference "C15")
+					(unit 1)
+				)
